Commit message: first commit

File: catkin_ws/src/simulation/walker_description/urdf/walker.urdf.xacro (robot description, xacro)
@@ -3,8 +3,10 @@
     <!-- <xacro:arg name="robot_namespace" default="/" />  -->
     <xacro:arg name="robot_namespace" default="walker" />
+    <xacro:arg name="realsense_enabled" default="1" />
     <!-- Included URDF/XACRO Files -->
     <xacro:include filename="$(find walker_description)/urdf/accessories/webcam_c930e.urdf.xacro"/>
     <xacro:include filename="$(find walker_description)/urdf/accessories/ydlidar_g4.urdf.xacro" />
     <xacro:include filename="$(find walker_description)/urdf/accessories/estop.urdf.xacro" />
+    <!-- <xacro:include filename="$(find walker_description)/urdf/accessories/intel_realsense.urdf.xacro"/> -->
     <!-- Gazebo plugin -->
     <xacro:include filename="$(find walker_description)/urdf/walker.gazebo" />
@@ -66,5 +68,5 @@
             <!-- <inertia ixx="0.00013887" ixy="-1.6386E-36" ixz="2.1452E-37"
                     iyy="0.00013887" iyz="-7.5427E-20" izz="0.00026251" /> -->
-            <cylinder_inertia m="${rear_wheel_mass}" r="${rear_wheel_radius}" h="${rear_wheel_width}" />
+            <xacro:cylinder_inertia m="${rear_wheel_mass}" r="${rear_wheel_radius}" h="${rear_wheel_width}" />
         </inertial>
         <visual>
@@ -103,5 +105,5 @@
             <!-- <inertia ixx="0.00013887" ixy="4.2884E-36" ixz="-8.5028E-20"
                     iyy="0.00013887" iyz="-7.5708E-21" izz="0.00026251" /> -->
-            <cylinder_inertia m="${rear_wheel_mass}" r="${rear_wheel_radius}" h="${rear_wheel_width}" />
+            <xacro:cylinder_inertia m="${rear_wheel_mass}" r="${rear_wheel_radius}" h="${rear_wheel_width}" />
         </inertial>
         <visual>
@@ -142,5 +144,5 @@
             <!-- <inertia ixx="8.7156E-05" ixy="-9.4168E-06" ixz="4.2663E-06"
                     iyy="0.00011084" iyz="1.6414E-06" izz="0.0001673" /> -->
-            <cylinder_inertia m="0.5" r="0.04" h="0.03" />
+            <xacro:cylinder_inertia m="0.5" r="0.04" h="0.03" />
         </inertial>
         <visual>
@@ -208,5 +210,5 @@
             <origin xyz="0 0 0" rpy="0 0 0" />
             <mass value="${front_wheel_mass}" />
-            <sphere_inertia m="${front_wheel_mass}" r="${front_wheel_radius}"/>
+            <xacro:sphere_inertia m="${front_wheel_mass}" r="${front_wheel_radius}"/>
         </inertial>
         <visual>
@@ -239,5 +241,5 @@
             <origin xyz="0 0 0" rpy="0 0 0" />
             <mass value="${front_wheel_mass}" />
-            <sphere_inertia m="${front_wheel_mass}" r="${front_wheel_radius}"/>
+            <xacro:sphere_inertia m="${front_wheel_mass}" r="${front_wheel_radius}"/>
         </inertial>
         <visual>
@@ -265,6 +267,17 @@
         <axis xyz="0 0 0" />
     </joint>
+    <!-- Intel realsense D435 -->
+    <xacro:if value="$(arg realsense_enabled)">
+    <xacro:include filename="$(find walker_description)/urdf/accessories/intel_realsense.urdf.xacro"/>
+        <xacro:intel_realsense_mount prefix="camera1" topic="camera1" parent_link="realsense_mount"/>
+        <link name="realsense_mount"/>
+        <joint name="realsense_mount_joint" type="fixed">
+        <origin xyz="0 0 0.012" rpy="0 0 ${-M_PI}" />
+        <parent link="laser_link"/>
+        <child link="realsense_mount" />
+        </joint>
+    </xacro:if>
     <!-- YDLiDAR G4 plugin -->
-    <ydlidar_g4 frame="laser" topic="scan" min_angle="${M_PI / 4}" max_angle="${M_PI / 4 * 7}" robot_namespace="$(arg robot_namespace)"/>
+    <xacro:ydlidar_g4 frame="laser" topic="scan" min_angle="${M_PI / 4}" max_angle="${M_PI / 4 * 7}" robot_namespace="$(arg robot_namespace)"/>
     <joint name="ydlidar_mount_joint" type="fixed">
         <origin xyz="${ydlidar_xyz}" rpy="${ydlidar_rpy}" />
@@ -273,5 +286,5 @@
     </joint>
     <!-- Logitech C930e webcam -->
-    <webcam_c930e frame="camera" topic="usb_cam" robot_namespace="$(arg robot_namespace)"/>
+    <xacro:webcam_c930e frame="camera" topic="usb_cam" robot_namespace="$(arg robot_namespace)"/>
     <joint name="webcam_mount_joint" type="fixed">
         <origin xyz="${webcam_xyz}" rpy="${webcam_rpy}" />
@@ -284,5 +297,5 @@
             <origin xyz="0.1 0 0" rpy="0 0 0" />
             <mass value="0.1" />
-            <box_inertia m="0.1" x="0.2" y="0.08" z="0.01"/>
+            <xacro:box_inertia m="0.1" x="0.2" y="0.08" z="0.01"/>
         </inertial>
         <collision name='collision'>
@@ -308,5 +321,5 @@
     </joint>
     <!-- E-stop -->
-    <estop frame="estop" />
+    <xacro:estop frame="estop" />
     <joint name="estop_joint1" type="fixed">
         <origin xyz="0.161 0 0.905" rpy="0 0 0" />
